Commit message: Progress towards simulated moveit without connection to the robot

File: ROS/src/mg400_ros2_bringup/config/mg400.urdf.xacro (robot description, xacro)
@@ -318,2 +318,9 @@
     />
 </robot>
+    <!-- <xacro:arg name="initial_positions_file" default="initial_positions.yaml" />
+    <!-- Import mg400 urdf file -->
+    <xacro:include filename="$(find mg400_ros2_bringup)/urdf/mg400.urdf.xacro" />
+    <!-- Import control_xacro -->
+    <xacro:include filename="mg400.ros2_control.xacro" />
+    <xacro:mg400_ros2_control name="FakeSystem" initial_positions_file="$(arg initial_positions_file)"/>
+</robot> -->

File: ROS/src/mg400_ros2_bringup/urdf/mg400.urdf.xacro (robot description, xacro)
@@ -1,3 +1,3 @@
-<?xml version="1.0"?>
+<?xml version="1.0" encoding="utf-8"?>
 <robot xmlns:xacro="http://www.ros.org/wiki/xacro" name="mg400">
     <!-- =================================================================================== -->
@@ -317,3 +317,9 @@
     j4_upper_limit="${j4_upper_limit}"
     />
+    <!-- <xacro:if value="$(arg use_mock)">
+        <xacro:mg400_mock_ros2_control/>
+    </xacro:if>
+    <xacro:unless value="$(arg use_mock)">
+        <xacro:mg400_ros2_control/>
+    </xacro:unless> -->
 </robot>

File: ROS/src/mg400_ros2_bringup/urdf/mg400_mock.ros2_control.xacro (robot description, xacro)
@@ -6,17 +6,10 @@
     The joint limit parameters are passed from the main URDF xacro.
   -->
-  <xacro:macro name="mg400_ros2_control" params="
-    j1_lower_limit
-    j1_upper_limit
-    j2_lower_limit
-    j2_upper_limit
-    j3_lower_limit
-    j3_upper_limit
-    j4_lower_limit
-    j4_upper_limit">
-    <ros2_control name="MG400SystemHardware" type="system">
+  <xacro:macro name="mg400_mock_ros2_control">
+    <ros2_control name="MockMG400" type="system">
       <hardware>
+        <plugin>mock_components/GenericSystem</plugin>
         <!-- This plugin connects ros2_control to the C++ hardware interface -->
-        <plugin>mg400_ros2_bringup/MG400SystemHardware</plugin>
+        <!-- <plugin>mg400_ros2_bringup/MockMG400SystemHardware</plugin> -->
       </hardware>
       <!-- Define the commandable joints for the controller manager -->
@@ -24,6 +17,6 @@
       <joint name="j1">
         <command_interface name="position">
-          <param name="min">${j1_lower_limit}</param>
-          <param name="max">${j1_upper_limit}</param>
+          <param name="min">${J1_MIN_RAD}</param>
+          <param name="max">${J1_MAX_RAD}</param>
         </command_interface>
         <command_interface name="velocity"/>
@@ -35,6 +28,6 @@
       <joint name="j2">
         <command_interface name="position">
-          <param name="min">${j2_lower_limit}</param>
-          <param name="max">${j2_upper_limit}</param>
+          <param name="min">${J2_MIN_RAD}</param>
+          <param name="max">${J2_MAX_RAD}</param>
         </command_interface>
         <command_interface name="velocity"/>
@@ -46,6 +39,6 @@
       <joint name="j3">
         <command_interface name="position">
-          <param name="min">${j3_lower_limit}</param>
-          <param name="max">${j3_upper_limit}</param>
+          <param name="min">${J3_MIN_RAD}</param>
+          <param name="max">${J3_MAX_RAD}</param>
         </command_interface>
         <command_interface name="velocity"/>
@@ -57,6 +50,6 @@
       <joint name="j4">
         <command_interface name="position">
-          <param name="min">${j4_lower_limit}</param>
-          <param name="max">${j4_upper_limit}</param>
+          <param name="min">${J4_MIN_RAD}</param>
+          <param name="max">${J4_MAX_RAD}</param>
         </command_interface>
         <command_interface name="velocity"/>
