Commit message: Added extra internal link to find more illegal states

File: ROS/src/mg400_ros2_bringup/config/mg400.ros2_control.xacro (robot description, xacro)
@@ -1,69 +1,40 @@
 <?xml version="1.0"?>
 <robot xmlns:xacro="http://www.ros.org/wiki/xacro">
-  <!--
-    This file defines the ros2_control interfaces for the MG400 robot.
-    It specifies the hardware plugin, the commandable joints, and their state interfaces.
-    The joint limit parameters are passed from the main URDF xacro.
-  -->
-  <xacro:macro name="mg400_ros2_control" params="
-    j1_lower_limit
-    j1_upper_limit
-    j2_lower_limit
-    j2_upper_limit
-    j3_lower_limit
-    j3_upper_limit
-    j4_lower_limit
-    j4_upper_limit">
-    <ros2_control name="MG400SystemHardware" type="system">
-      <hardware>
-        <!-- This plugin connects ros2_control to the C++ hardware interface -->
-        <plugin>mg400_ros2_bringup/MG400SystemHardware</plugin>
-      </hardware>
-      <!-- Define the commandable joints for the controller manager -->
-      <!-- Joint 1 -->
-      <joint name="j1">
-        <command_interface name="position">
-          <param name="min">${j1_lower_limit}</param>
-          <param name="max">${j1_upper_limit}</param>
-        </command_interface>
-        <command_interface name="velocity"/>
-        <command_interface name="acceleration"/>
-        <state_interface name="position"/>
-        <state_interface name="velocity"/>
-      </joint>
-      <!-- Joint 2 -->
-      <joint name="j2">
-        <command_interface name="position">
-          <param name="min">${j2_lower_limit}</param>
-          <param name="max">${j2_upper_limit}</param>
-        </command_interface>
-        <command_interface name="velocity"/>
-        <command_interface name="acceleration"/>
-        <state_interface name="position"/>
-        <state_interface name="velocity"/>
-      </joint>
-      <!-- Joint 3 -->
-      <joint name="j3">
-        <command_interface name="position">
-          <param name="min">${j3_lower_limit}</param>
-          <param name="max">${j3_upper_limit}</param>
-        </command_interface>
-        <command_interface name="velocity"/>
-        <command_interface name="acceleration"/>
-        <state_interface name="position"/>
-        <state_interface name="velocity"/>
-      </joint>
-      <!-- Joint 4 -->
-      <joint name="j4">
-        <command_interface name="position">
-          <param name="min">${j4_lower_limit}</param>
-          <param name="max">${j4_upper_limit}</param>
-        </command_interface>
-        <command_interface name="velocity"/>
-        <command_interface name="acceleration"/>
-        <state_interface name="position"/>
-        <state_interface name="velocity"/>
-      </joint>
-    </ros2_control>
-  </xacro:macro>
+    <xacro:macro name="mg400_ros2_control" params="name initial_positions_file">
+        <xacro:property name="initial_positions" value="${xacro.load_yaml(initial_positions_file)['initial_positions']}"/>
+        <ros2_control name="${name}" type="system">
+            <hardware>
+                <!-- By default, set up controllers for simulation. This won't work on real hardware -->
+                <plugin>mock_components/GenericSystem</plugin>
+            </hardware>
+            <joint name="j1">
+                <command_interface name="position"/>
+                <state_interface name="position">
+                  <param name="initial_value">${initial_positions['j1']}</param>
+                </state_interface>
+                <state_interface name="velocity"/>
+            </joint>
+            <joint name="j2">
+                <command_interface name="position"/>
+                <state_interface name="position">
+                  <param name="initial_value">${initial_positions['j2']}</param>
+                </state_interface>
+                <state_interface name="velocity"/>
+            </joint>
+            <joint name="j3">
+                <command_interface name="position"/>
+                <state_interface name="position">
+                  <param name="initial_value">${initial_positions['j3']}</param>
+                </state_interface>
+                <state_interface name="velocity"/>
+            </joint>
+            <joint name="j4">
+                <command_interface name="position"/>
+                <state_interface name="position">
+                  <param name="initial_value">${initial_positions['j4']}</param>
+                </state_interface>
+                <state_interface name="velocity"/>
+            </joint>
+        </ros2_control>
+    </xacro:macro>
 </robot>

File: ROS/src/mg400_ros2_bringup/config/mg400.urdf.xacro (robot description, xacro)
@@ -1,322 +1,5 @@
 <?xml version="1.0"?>
 <robot xmlns:xacro="http://www.ros.org/wiki/xacro" name="mg400">
-    <!-- =================================================================================== -->
-    <!-- |                                  PROPERTIES                                     | -->
-    <!-- =================================================================================== -->
-    <!-- Constants -->
-    <xacro:property name="PI" value="3.1415926535897931"/>
-    <xacro:property name="deg_to_rad" value="${PI / 180.0}"/>
-    <!-- Base path for mesh files -->
-    <xacro:property name="BASE_PATH" value="package://mg400_ros2_bringup/urdf/meshes"/>
-    <!-- Joint Limits from Manual (Appendix A, page 41) -->
-    <!-- Position Limits (rad) -->
-    <xacro:property name="j1_lower_limit" value="${-160 * deg_to_rad}"/>
-    <xacro:property name="j1_upper_limit" value="${160 * deg_to_rad}"/>
-    <xacro:property name="j2_lower_limit" value="${-25 * deg_to_rad}"/>
-    <xacro:property name="j2_upper_limit" value="${85 * deg_to_rad}"/>
-    <xacro:property name="j3_lower_limit" value="${-25 * deg_to_rad}"/>
-    <xacro:property name="j3_upper_limit" value="${105 * deg_to_rad}"/>
-    <xacro:property name="j4_lower_limit" value="${-360 * deg_to_rad}"/>
-    <xacro:property name="j4_upper_limit" value="${360 * deg_to_rad}"/>
-    <!-- Velocity Limits (rad/s) -->
-    <xacro:property name="j_velocity_limit" value="${300 * deg_to_rad}"/>
-    <!-- Joint Origins -->
-    <xacro:property name="j1_xyz" value="-0.005 0 0.109"/>
-    <xacro:property name="j2_xyz" value="0.0435007595118091 -0.0357748756218899 0.118995682641123"/>
-    <xacro:property name="j3_xyz" value="-0.0010512570171516 0.0357748756218898 0.175001164344716"/>
-    <xacro:property name="j4_1_xyz" value="0.174969784055705 -0.0170000000000335 0.00325187137614585"/>
-    <xacro:property name="j4_xyz" value="0.0659996239003897 0.0170000000000371 0.031000800715573"/>
-    <xacro:property name="j2_2_xyz" value="0.00452885682964267 -0.0305 0.141500000000001"/>
-    <xacro:property name="j3_2_xyz" value="-0.00105049750546494 0.00649999999999986 0.174996846985851"/>
-    <xacro:property name="j4_2_xyz" value="0.0678965856063864 0.000500000000000073 0.0119719999403219"/>
-    <!-- Import ros2_control configuration -->
-    <xacro:include filename="$(find mg400_ros2_bringup)/urdf/mg400.ros2_control.xacro" />
-    <!-- =================================================================================== -->
-    <!-- |                                     ROBOT                                       | -->
-    <!-- =================================================================================== -->
-    <link name="base_link">
-        <inertial>
-            <origin xyz="0.000600637001378879 -2.53487071137343E-07 0.0560927888040551" rpy="0 0 0"/>
-            <mass value="3.62164811695094"/>
-            <inertia ixx="0.0126582175296405" ixy="6.66832041405407E-08" ixz="-3.52548281362717E-06" iyy="0.0145891535260188" iyz="5.15901657460475E-08" izz="0.0195045116656827"/>
-        </inertial>
-        <visual>
-            <origin xyz="0 0 0" rpy="0 0 0"/>
-            <geometry>
-                <mesh filename="${BASE_PATH}/base_link.STL"/>
-            </geometry>
-            <material name="">
-                <color rgba="1 1 1 1"/>
-            </material>
-        </visual>
-        <collision>
-            <origin xyz="0 0 0" rpy="0 0 0"/>
-            <geometry>
-                <mesh filename="${BASE_PATH}/base_link.STL"/>
-            </geometry>
-        </collision>
-    </link>
-    <link name="link1">
-        <inertial>
-            <origin xyz="-0.0046209286967387 -6.88107982318643E-05 0.0709919358465827" rpy="0 0 0"/>
-            <mass value="1.77056222753813"/>
-            <inertia ixx="0.00605885293080088" ixy="0.000156081820035162" ixz="-0.00021785654850453" iyy="0.00579381982249127" iyz="6.20876898015621E-05" izz="0.00741058257251941"/>
-        </inertial>
-        <visual>
-            <origin xyz="0 0 0" rpy="0 0 0"/>
-            <geometry>
-                <mesh filename="${BASE_PATH}/link1.STL"/>
-            </geometry>
-            <material name="">
-                <color rgba="1 1 1 1"/>
-            </material>
-        </visual>
-        <collision>
-            <origin xyz="0 0 0" rpy="0 0 0"/>
-            <geometry>
-                <mesh filename="${BASE_PATH}/link1.STL"/>
-            </geometry>
-        </collision>
-    </link>
-    <joint name="j1" type="revolute">
-        <origin xyz="${j1_xyz}" rpy="0 0 0"/>
-        <parent link="base_link"/>
-        <child link="link1"/>
-        <axis xyz="0 0 1"/>
-        <limit lower="${j1_lower_limit}" upper="${j1_upper_limit}" effort="100" velocity="${j_velocity_limit}"/>
-    </joint>
-    <!-- Main kinematic chain -->
-    <link name="link2_1">
-        <inertial>
-            <origin xyz="-0.00321788524756698 0.0352926570826593 0.0596131328734945" rpy="0 0 0"/>
-            <mass value="0.0866115884541459"/>
-            <inertia ixx="0.000338551627157209" ixy="-2.78858228577314E-09" ixz="1.05212346076681E-05" iyy="0.000307789653713489" iyz="-1.36109590152488E-06" izz="3.89949940178023E-05"/>
-        </inertial>
-        <visual>
-            <origin xyz="0 0 0" rpy="0 0 0"/>
-            <geometry>
-                <mesh filename="${BASE_PATH}/link2_1.STL"/>
-            </geometry>
-            <material name="">
-                <color rgba="1 1 1 1"/>
-            </material>
-        </visual>
-        <collision>
-            <origin xyz="0 0 0" rpy="0 0 0"/>
-            <geometry>
-                <mesh filename="${BASE_PATH}/link2_1.STL"/>
-            </geometry>
-        </collision>
-    </link>
-    <joint name="j2" type="revolute">
-        <origin xyz="${j2_xyz}" rpy="0 0 0"/>
-        <parent link="link1"/>
-        <child link="link2_1"/>
-        <axis xyz="0 1 0"/>
-        <limit lower="${j2_lower_limit}" upper="${j2_upper_limit}" effort="100" velocity="${j_velocity_limit}"/>
-    </joint>
-    <link name="link3_1">
-        <inertial>
-            <origin xyz="0.0821679417596488 0.000113044685842874 -0.00333758753063973" rpy="0 0 0"/>
-            <mass value="0.0375214831045061"/>
-            <inertia ixx="2.54761091812684E-06" ixy="3.73102654491378E-07" ixz="-2.02625705871199E-06" iyy="0.000164234314177935" iyz="-1.44731096825347E-08" izz="0.000164331500854172"/>
-        </inertial>
-        <visual>
-            <origin xyz="0 0 0" rpy="0 0 0"/>
-            <geometry>
-                <mesh filename="${BASE_PATH}/link3_1.STL"/>
-            </geometry>
-            <material name="">
-                <color rgba="1 1 1 1"/>
-            </material>
-        </visual>
-        <collision>
-            <origin xyz="0 0 0" rpy="0 0 0"/>
-            <geometry>
-                <mesh filename="${BASE_PATH}/link3_1.STL"/>
-            </geometry>
-        </collision>
-    </link>
-    <!-- The fake_link is an intermediate frame to correctly model the parallelogram linkage -->
-    <link name="fake_link" />
-    <joint name="j3" type="revolute">
-        <origin xyz="${j3_xyz}" rpy="0 0 0"/>
-        <parent link="link2_1"/>
-        <child link="fake_link"/>
-        <axis xyz="0 1 0"/>
-        <limit lower="${j3_lower_limit}" upper="${j3_upper_limit}" effort="100" velocity="${j_velocity_limit}"/>
-    </joint>
-    <joint name="j3_1" type="revolute">
-        <origin xyz="0 0 0" rpy="0 0 0"/>
-        <parent link="fake_link"/>
-        <child link="link3_1"/>
-        <axis xyz="0 1 0"/>
-        <limit lower="${-PI}" upper="${PI}" effort="0" velocity="${j_velocity_limit}"/>
-        <mimic joint="j3_2" />
-    </joint>
-    <link name="link4_1">
-        <inertial>
-            <origin xyz="0.0387878182928232 0.0170848333998282 -0.0024610990490942" rpy="0 0 0"/>
-            <mass value="0.0628979533925801"/>
-            <inertia ixx="4.78483605712844E-05" ixy="1.42081909356751E-07" ixz="8.32917079044309E-06" iyy="5.42362047732042E-05" iyz="-2.90608446019989E-08" izz="3.36120409842199E-05"/>
-        </inertial>
-        <visual>
-            <origin xyz="0 0 0" rpy="0 0 0"/>
-            <geometry>
-                <mesh filename="${BASE_PATH}/link4_1.STL"/>
-            </geometry>
-            <material name="">
-                <color rgba="1 1 1 1"/>
-            </material>
-        </visual>
-        <collision>
-            <origin xyz="0 0 0" rpy="0 0 0"/>
-            <geometry>
-                <mesh filename="${BASE_PATH}/link4_1.STL"/>
-            </geometry>
-        </collision>
-    </link>
-    <joint name="j4_1" type="revolute">
-        <origin xyz="${j4_1_xyz}" rpy="0 0 0"/>
-        <parent link="link3_1"/>
-        <child link="link4_1"/>
-        <axis xyz="0 1 0"/>
-        <limit lower="${-PI}" upper="${PI}" effort="0" velocity="${j_velocity_limit}"/>
-        <mimic joint="j4_2" multiplier="-1" />
-    </joint>
-    <link name="link5">
-        <inertial>
-            <origin xyz="4.24246458685662E-07 3.08507851181768E-14 -0.0349688816440933" rpy="0 0 0"/>
-            <mass value="0.0965276919819365"/>
-            <inertia ixx="4.98589992160928E-05" ixy="-1.534865545378E-12" ixz="3.46424449605658E-10" iyy="4.98589881725446E-05" iyz="-5.64890953414983E-17" izz="2.130463008359E-05"/>
-        </inertial>
-        <visual>
-            <origin xyz="0 0 0" rpy="0 0 0"/>
-            <geometry>
-                <mesh filename="${BASE_PATH}/link5.STL"/>
-            </geometry>
-            <material name="">
-                <color rgba="1 1 1 1"/>
-            </material>
-        </visual>
-        <collision>
-            <origin xyz="0 0 0" rpy="0 0 0"/>
-            <geometry>
-                <mesh filename="${BASE_PATH}/link5.STL"/>
-            </geometry>
-        </collision>
-    </link>
-    <joint name="j4" type="revolute">
-        <origin xyz="${j4_xyz}" rpy="0 0 0"/>
-        <parent link="link4_1"/>
-        <child link="link5"/>
-        <!-- Axis is almost [0, 0, 1] -->
-        <axis xyz="-1.19408295462994E-05 0 0.999999999928708"/>
-        <limit lower="${j4_lower_limit}" upper="${j4_upper_limit}" effort="100" velocity="${j_velocity_limit}"/>
-    </joint>
-    <!-- Parallel linkage chain -->
-    <link name="link2_2">
-        <inertial>
-            <origin xyz="-0.0201111131723385 0.0304999635268521 0.073632809340276" rpy="0 0 0"/>
-            <mass value="0.0662546292985346"/>
-            <inertia ixx="0.000218973873589181" ixy="3.0147933007673E-10" ixz="2.51402553227571E-06" iyy="0.000200510070261609" iyz="-1.41837669904595E-09" izz="3.74316777806776E-05"/>
-        </inertial>
-        <visual>
-            <origin xyz="0 0 0" rpy="0 0 0"/>
-            <geometry>
-                <mesh filename="${BASE_PATH}/link2_2.STL"/>
-            </geometry>
-            <material name="">
-                <color rgba="1 1 1 1"/>
-            </material>
-        </visual>
-        <collision>
-            <origin xyz="0 0 0" rpy="0 0 0"/>
-            <geometry>
-                <mesh filename="${BASE_PATH}/link2_2.STL"/>
-            </geometry>
-        </collision>
-    </link>
-    <joint name="j2_2" type="revolute">
-        <origin xyz="${j2_2_xyz}" rpy="0 0 0"/>
-        <parent link="link1"/>
-        <child link="link2_2"/>
-        <axis xyz="0 1 0"/>
-        <limit lower="${-PI}" upper="${PI}" effort="0" velocity="${j_velocity_limit}"/>
-        <mimic joint="j2" />
-    </joint>
-    <link name="link3_2">
-        <inertial>
-            <origin xyz="0.0338566736074436 0.0240208873857428 0.00452229895926692" rpy="0 0 0"/>
-            <mass value="0.0366692789294813"/>
-            <inertia ixx="7.24011830695354E-06" ixy="7.93542746250724E-10" ixz="-1.69163254472566E-06" iyy="2.34967008246727E-05" iyz="4.55507111386579E-10" izz="1.66831643179488E-05"/>
-        </inertial>
-        <visual>
-            <origin xyz="0 0 0" rpy="0 0 0"/>
-            <geometry>
-                <mesh filename="${BASE_PATH}/link3_2.STL"/>
-            </geometry>
-            <material name="">
-                <color rgba="1 1 1 1"/>
-            </material>
-        </visual>
-        <collision>
-            <origin xyz="0 0 0" rpy="0 0 0"/>
-            <geometry>
-                <mesh filename="${BASE_PATH}/link3_2.STL"/>
-            </geometry>
-        </collision>
-    </link>
-    <joint name="j3_2" type="revolute">
-        <origin xyz="${j3_2_xyz}" rpy="0 0 0"/>
-        <parent link="link2_2"/>
-        <child link="link3_2"/>
-        <axis xyz="0 1 0"/>
-        <limit lower="${-PI}" upper="${PI}" effort="0" velocity="${j_velocity_limit}"/>
-        <mimic joint="j2_2" multiplier="-1" />
-    </joint>
-    <link name="link4_2">
-        <inertial>
-            <origin xyz="0.0876391591012518 0.023499867452275 0.00831492252441945" rpy="0 0 0"/>
-            <mass value="0.0453569016333092"/>
-            <inertia ixx="2.00037596001325E-05" ixy="3.34474706250153E-09" ixz="2.17594982354756E-07" iyy="0.000132049841023893" iyz="5.36978669669685E-10" izz="0.000141813978894428"/>
-        </inertial>
-        <visual>
-            <origin xyz="0 0 0" rpy="0 0 0"/>
-            <geometry>
-                <mesh filename="${BASE_PATH}/link4_2.STL"/>
-            </geometry>
-            <material name="">
-                <color rgba="1 1 1 1"/>
-            </material>
-        </visual>
-        <collision>
-            <origin xyz="0 0 0" rpy="0 0 0"/>
-            <geometry>
-                <mesh filename="${BASE_PATH}/link4_2.STL"/>
-            </geometry>
-        </collision>
-    </link>
-    <joint name="j4_2" type="revolute">
-        <origin xyz="${j4_2_xyz}" rpy="0 0 0"/>
-        <parent link="link3_2"/>
-        <child link="link4_2"/>
-        <axis xyz="0 1 0"/>
-        <limit lower="${-PI}" upper="${PI}" effort="0" velocity="${j_velocity_limit}"/>
-        <mimic joint="j3"/>
-    </joint>
-    <!-- Instantiate ros2_control plugin -->
-    <xacro:mg400_ros2_control
-    j1_lower_limit="${j1_lower_limit}"
-    j1_upper_limit="${j1_upper_limit}"
-    j2_lower_limit="${j2_lower_limit}"
-    j2_upper_limit="${j2_upper_limit}"
-    j3_lower_limit="${j3_lower_limit}"
-    j3_upper_limit="${j3_upper_limit}"
-    j4_lower_limit="${j4_lower_limit}"
-    j4_upper_limit="${j4_upper_limit}"
-    />
-</robot>
-    <!-- <xacro:arg name="initial_positions_file" default="initial_positions.yaml" />
+    <xacro:arg name="initial_positions_file" default="initial_positions.yaml" />
     <!-- Import mg400 urdf file -->
     <xacro:include filename="$(find mg400_ros2_bringup)/urdf/mg400.urdf.xacro" />
@@ -324,3 +7,3 @@
     <xacro:include filename="mg400.ros2_control.xacro" />
     <xacro:mg400_ros2_control name="FakeSystem" initial_positions_file="$(arg initial_positions_file)"/>
-</robot> -->
+</robot>

File: ROS/src/mg400_ros2_bringup/urdf/mg400.urdf.xacro (robot description, xacro)
@@ -28,4 +28,5 @@
     <xacro:property name="j4_xyz" value="0.0659996239003897 0.0170000000000371 0.031000800715573"/>
     <xacro:property name="j2_2_xyz" value="0.00452885682964267 -0.0305 0.141500000000001"/>
+    <xacro:property name="j2_3_xyz" value="-0.043 0.0 0.0"/>
     <xacro:property name="j3_2_xyz" value="-0.00105049750546494 0.00649999999999986 0.174996846985851"/>
     <xacro:property name="j4_2_xyz" value="0.0678965856063864 0.000500000000000073 0.0119719999403219"/>
@@ -154,5 +155,5 @@
         <axis xyz="0 1 0"/>
         <limit lower="${-PI}" upper="${PI}" effort="0" velocity="${j_velocity_limit}"/>
-        <mimic joint="j3_2" />
+        <mimic joint="j2" multiplier="-1" />
     </joint>
     <link name="link4_1">
@@ -184,5 +185,5 @@
         <axis xyz="0 1 0"/>
         <limit lower="${-PI}" upper="${PI}" effort="0" velocity="${j_velocity_limit}"/>
-        <mimic joint="j4_2" multiplier="-1" />
+        <mimic joint="j3" multiplier="-1" />
     </joint>
     <link name="link5">
@@ -247,4 +248,47 @@
         <mimic joint="j2" />
     </joint>
+    <!-- Parallel linkage chain in between outer and inner link-->
+    <!-- TODO: Mass is just a random guess -->
+    <link name="link2_3">
+        <inertial>
+            <origin xyz="0.0 0.0 0.0" rpy="0 0 0"/>
+            <mass value="0.0062546292985346"/>
+            <inertia ixx="0.000218973873589181" ixy="3.0147933007673E-10" ixz="2.51402553227571E-06" iyy="0.000200510070261609" iyz="-1.41837669904595E-09" izz="3.74316777806776E-05"/>
+        </inertial>
+        <visual>
+            <origin xyz="0.001 -0.0035 -0.086" rpy="0 0 0"/>
+            <geometry>
+                <box size="0.008 0.005 0.174"/>
+            </geometry>
+            <material name="">
+                <color rgba="0.5 0.5 0 1"/>
+            </material>
+        </visual>
+        <!-- [x] 1mm larger per side collision  -->
+        <collision>
+            <origin xyz="0.002 -0.0036 -0.086" rpy="0 0 0"/>
+            <geometry>
+                <box size="0.010 0.005 0.174"/>
+            </geometry>
+        </collision>
+    </link>
+    <!-- The fake_link is an intermediate frame to correctly model the parallelogram linkage -->
+    <link name="fake_link_2" />
+    <joint name="j2_3" type="revolute">
+        <origin xyz="${j2_3_xyz}" rpy="0 0 0"/>
+        <parent link="link3_1"/>
+        <child link="fake_link_2"/>
+        <axis xyz="0 1 0"/>
+        <limit lower="${-PI}" upper="${PI}" effort="0" velocity="${j_velocity_limit}"/>
+        <mimic joint="j2" />
+    </joint>
+    <joint name="j2_4" type="revolute">
+        <origin xyz="0 0 0" rpy="0 0 0"/>
+        <parent link="fake_link_2"/>
+        <child link="link2_3"/>
+        <axis xyz="0 1 0"/>
+        <limit lower="${-PI}" upper="${PI}" effort="0" velocity="${j_velocity_limit}"/>
+        <mimic joint="j3" multiplier="-1"/>
+    </joint>
     <link name="link3_2">
         <inertial>
@@ -275,5 +319,5 @@
         <axis xyz="0 1 0"/>
         <limit lower="${-PI}" upper="${PI}" effort="0" velocity="${j_velocity_limit}"/>
-        <mimic joint="j2_2" multiplier="-1" />
+        <mimic joint="j2" multiplier="-1" />
     </joint>
     <link name="link4_2">
