Commit message: fixes to last merge for program to boot. Thinks its fine :)

File: ROS/src/mg400_ros2_bringup/urdf/mg400.urdf.xacro (robot description, xacro)
@@ -32,4 +32,5 @@
     <!-- Import ros2_control configuration -->
     <xacro:include filename="$(find mg400_ros2_bringup)/urdf/mg400.ros2_control.xacro" />
+    <xacro:include filename="$(find mg400_ros2_bringup)/urdf/mg400_mock.ros2_control.xacro" />
     <!-- =================================================================================== -->
     <!-- |                                     ROBOT                                       | -->
@@ -317,9 +318,27 @@
     j4_upper_limit="${j4_upper_limit}"
     />
-    <!-- <xacro:if value="$(arg use_mock)">
-        <xacro:mg400_mock_ros2_control/>
+    <xacro:if value="$(arg use_mock)">
+        <xacro:mg400_mock_ros2_control
+        j1_lower_limit="${j1_lower_limit}"
+        j1_upper_limit="${j1_upper_limit}"
+        j2_lower_limit="${j2_lower_limit}"
+        j2_upper_limit="${j2_upper_limit}"
+        j3_lower_limit="${j3_lower_limit}"
+        j3_upper_limit="${j3_upper_limit}"
+        j4_lower_limit="${j4_lower_limit}"
+        j4_upper_limit="${j4_upper_limit}"
+        />
     </xacro:if>
     <xacro:unless value="$(arg use_mock)">
-        <xacro:mg400_ros2_control/>
-    </xacro:unless> -->
+        <xacro:mg400_ros2_control
+        j1_lower_limit="${j1_lower_limit}"
+        j1_upper_limit="${j1_upper_limit}"
+        j2_lower_limit="${j2_lower_limit}"
+        j2_upper_limit="${j2_upper_limit}"
+        j3_lower_limit="${j3_lower_limit}"
+        j3_upper_limit="${j3_upper_limit}"
+        j4_lower_limit="${j4_lower_limit}"
+        j4_upper_limit="${j4_upper_limit}"
+        />
+    </xacro:unless>
 </robot>

File: ROS/src/mg400_ros2_bringup/urdf/mg400_mock.ros2_control.xacro (robot description, xacro)
@@ -6,10 +6,18 @@
     The joint limit parameters are passed from the main URDF xacro.
   -->
-  <xacro:macro name="mg400_mock_ros2_control">
+  <xacro:macro name="mg400_mock_ros2_control" params="
+    j1_lower_limit
+    j1_upper_limit
+    j2_lower_limit
+    j2_upper_limit
+    j3_lower_limit
+    j3_upper_limit
+    j4_lower_limit
+    j4_upper_limit
+  ">
     <ros2_control name="MockMG400" type="system">
       <hardware>
+        <!-- This plugin connects ros2_control to a mock hardware interface -->
         <plugin>mock_components/GenericSystem</plugin>
-        <!-- This plugin connects ros2_control to the C++ hardware interface -->
-        <!-- <plugin>mg400_ros2_bringup/MockMG400SystemHardware</plugin> -->
       </hardware>
       <!-- Define the commandable joints for the controller manager -->
@@ -17,6 +25,6 @@
       <joint name="j1">
         <command_interface name="position">
-          <param name="min">${J1_MIN_RAD}</param>
-          <param name="max">${J1_MAX_RAD}</param>
+          <param name="min">${j1_lower_limit}</param>
+          <param name="max">${j1_upper_limit}</param>
         </command_interface>
         <command_interface name="velocity"/>
@@ -28,6 +36,6 @@
       <joint name="j2">
         <command_interface name="position">
-          <param name="min">${J2_MIN_RAD}</param>
-          <param name="max">${J2_MAX_RAD}</param>
+          <param name="min">${j2_lower_limit}</param>
+          <param name="max">${j2_upper_limit}</param>
         </command_interface>
         <command_interface name="velocity"/>
@@ -39,6 +47,6 @@
       <joint name="j3">
         <command_interface name="position">
-          <param name="min">${J3_MIN_RAD}</param>
-          <param name="max">${J3_MAX_RAD}</param>
+          <param name="min">${j3_lower_limit}</param>
+          <param name="max">${j3_upper_limit}</param>
         </command_interface>
         <command_interface name="velocity"/>
@@ -50,6 +58,6 @@
       <joint name="j4">
         <command_interface name="position">
-          <param name="min">${J4_MIN_RAD}</param>
-          <param name="max">${J4_MAX_RAD}</param>
+          <param name="min">${j4_lower_limit}</param>
+          <param name="max">${j4_upper_limit}</param>
         </command_interface>
         <command_interface name="velocity"/>

Commit message: more conservative collision limits

File: ROS/src/mg400_ros2_bringup/urdf/mg400.urdf.xacro (robot description, xacro)
@@ -11,12 +11,12 @@
     <!-- Joint Limits from Manual (Appendix A, page 41) -->
     <!-- Position Limits (rad) -->
-    <xacro:property name="j1_lower_limit" value="${-160 * deg_to_rad}"/>
-    <xacro:property name="j1_upper_limit" value="${160 * deg_to_rad}"/>
-    <xacro:property name="j2_lower_limit" value="${-25 * deg_to_rad}"/>
-    <xacro:property name="j2_upper_limit" value="${85 * deg_to_rad}"/>
-    <xacro:property name="j3_lower_limit" value="${-25 * deg_to_rad}"/>
-    <xacro:property name="j3_upper_limit" value="${105 * deg_to_rad}"/>
-    <xacro:property name="j4_lower_limit" value="${-360 * deg_to_rad}"/>
-    <xacro:property name="j4_upper_limit" value="${360 * deg_to_rad}"/>
+    <xacro:property name="j1_lower_limit" value="${-158 * deg_to_rad}"/> <!-- Original limit: -160 -->
+    <xacro:property name="j1_upper_limit" value="${158 * deg_to_rad}"/> <!-- Original limit: 160 -->
+    <xacro:property name="j2_lower_limit" value="${-23 * deg_to_rad}"/> <!-- Original limit: -25 -->
+    <xacro:property name="j2_upper_limit" value="${83 * deg_to_rad}"/> <!-- Original limit: 85 -->
+    <xacro:property name="j3_lower_limit" value="${-23 * deg_to_rad}"/> <!-- Original limit: -25 -->
+    <xacro:property name="j3_upper_limit" value="${103 * deg_to_rad}"/> <!-- Original limit: 105 -->
+    <xacro:property name="j4_lower_limit" value="${-358 * deg_to_rad}"/> <!-- Original limit: -360 -->
+    <xacro:property name="j4_upper_limit" value="${358 * deg_to_rad}"/> <!-- Original limit: 360 -->
     <!-- Velocity Limits (rad/s) -->
     <xacro:property name="j_velocity_limit" value="${300 * deg_to_rad}"/>
@@ -264,7 +264,7 @@
         <!-- [x] 1mm larger per side collision  -->
         <collision>
-            <origin xyz="0.002 -0.0036 -0.086" rpy="0 0 0"/>
-            <geometry>
-                <box size="0.010 0.005 0.174"/>
+            <origin xyz="0.000 -0.0036 -0.086" rpy="0 0 0"/>
+            <geometry>
+                <box size="0.024 0.005 0.174"/>
             </geometry>
         </collision>

Commit message: Small edits to moveit config as well as the srdf. * Joints instead of chain * stomp as planer * no inertial on baselink

File: ROS/src/mg400_ros2_bringup/urdf/mg400.urdf.xacro (robot description, xacro)
@@ -35,9 +35,9 @@
     <!-- =================================================================================== -->
     <link name="base_link">
-        <inertial>
+        <!-- <inertial>
             <origin xyz="0.000600637001378879 -2.53487071137343E-07 0.0560927888040551" rpy="0 0 0"/>
             <mass value="3.62164811695094"/>
             <inertia ixx="0.0126582175296405" ixy="6.66832041405407E-08" ixz="-3.52548281362717E-06" iyy="0.0145891535260188" iyz="5.15901657460475E-08" izz="0.0195045116656827"/>
-        </inertial>
+        </inertial> -->
         <visual>
             <origin xyz="0 0 0" rpy="0 0 0"/>

Commit message: Refactor robot configuration: update author details, add support for end effector components and modifyed joints

File: ROS/src/mg400_ros2_bringup/urdf/mg400.urdf.xacro (robot description, xacro)
@@ -26,5 +26,5 @@
     <xacro:property name="j3_xyz" value="-0.0010512570171516 0.0357748756218898 0.175001164344716"/>
     <xacro:property name="j4_1_xyz" value="0.174969784055705 -0.0170000000000335 0.00325187137614585"/>
-    <xacro:property name="j4_xyz" value="0.0659996239003897 0.0170000000000371 0.031000800715573"/>
+    <xacro:property name="j4_3_xyz" value="0.0659996239003897 0.0170000000000371 0.031000800715573"/>
     <xacro:property name="j2_2_xyz" value="0.00452885682964267 -0.0305 0.141500000000001"/>
     <xacro:property name="j2_3_xyz" value="-0.043 0.0 0.0"/>
@@ -206,11 +206,9 @@
         </collision>
     </link>
-    <joint name="j4" type="revolute">
-        <origin xyz="${j4_xyz}" rpy="0 0 0"/>
+    <joint name="j4_3" type="fixed">
+        <origin xyz="${j4_3_xyz}" rpy="0 0 0"/>
         <parent link="link4_1"/>
         <child link="link5"/>
-        <!-- Axis is almost [0, 0, 1] -->
-        <axis xyz="-1.19408295462994E-05 0 0.999999999928708"/>
-        <limit lower="${j4_lower_limit}" upper="${j4_upper_limit}" effort="100" velocity="${j_velocity_limit}"/>
+        <axis xyz="0 1 0"/>
     </joint>
     <!-- Parallel linkage chain -->
@@ -348,3 +346,45 @@
         <mimic joint="j3"/>
     </joint>
+    <link name="end_effector_mount"/>
+    <joint name="j4" type="revolute">
+        <origin xyz="0 0 -0.085" rpy="0 0 0"/>
+        <parent link="link5"/>
+        <child link="end_effector_mount"/>
+        <!-- Axis is almost [0, 0, 1] -->
+        <axis xyz="-1.19408295462994E-05 0 0.999999999928708"/>
+        <limit lower="${j4_lower_limit}" upper="${j4_upper_limit}" effort="100" velocity="${j_velocity_limit}"/>
+    </joint>
+    <!-- TODO: mass is a guess from thin air -->
+    <link name="end_effector_laser_test">
+        <inertial>
+            <origin xyz="0.0 0.0 0.0" rpy="0 0 0"/>
+            <mass value="0.0012546292985346"/>
+            <inertia ixx="0.000218973873589181" ixy="3.0147933007673E-10" ixz="2.51402553227571E-06" iyy="0.000200510070261609" iyz="-1.41837669904595E-09" izz="3.74316777806776E-05"/>
+        </inertial>
+        <visual>
+            <!-- origin -lenght/2 + 5 -->
+            <origin xyz="0.0 0.0 -0.008" rpy="0 0 0"/>
+            <geometry>
+                <cylinder radius="0.008" length="0.026"/>
+            </geometry>
+            <material name="">
+                <color rgba="0.5 0.5 0 1"/>
+            </material>
+        </visual>
+        <!-- [x] 1mm larger diameter -->
+        <collision>
+            <!-- origin -lenght/2 + 5 + 6 -->
+            <origin xyz="0.0 0.0 -0.010" rpy="0 0 0"/>
+            <geometry>
+                <cylinder radius="0.009" length="0.038"/>
+            </geometry>
+        </collision>
+    </link>
+    <!-- To place it at the end but unsure if that is correct for an end_effector -->
+    <joint name="tool_joint" type="fixed">
+        <origin xyz="0 0 0" rpy="0 0 0"/>
+        <parent link="end_effector_mount"/>
+        <child link="end_effector_laser_test"/>
+        <axis xyz="0 0 1"/>
+    </joint>
 </robot>

Commit message: unknown error -2 from robot during execution

File: ROS/src/mg400_ros2_bringup/urdf/mg400.urdf.xacro (robot description, xacro)
@@ -11,12 +11,12 @@
     <!-- Joint Limits from Manual (Appendix A, page 41) -->
     <!-- Position Limits (rad) -->
-    <xacro:property name="j1_lower_limit" value="${-158 * deg_to_rad}"/> <!-- Original limit: -160 -->
-    <xacro:property name="j1_upper_limit" value="${158 * deg_to_rad}"/> <!-- Original limit: 160 -->
-    <xacro:property name="j2_lower_limit" value="${-23 * deg_to_rad}"/> <!-- Original limit: -25 -->
-    <xacro:property name="j2_upper_limit" value="${83 * deg_to_rad}"/> <!-- Original limit: 85 -->
-    <xacro:property name="j3_lower_limit" value="${-23 * deg_to_rad}"/> <!-- Original limit: -25 -->
-    <xacro:property name="j3_upper_limit" value="${103 * deg_to_rad}"/> <!-- Original limit: 105 -->
-    <xacro:property name="j4_lower_limit" value="${-358 * deg_to_rad}"/> <!-- Original limit: -360 -->
-    <xacro:property name="j4_upper_limit" value="${358 * deg_to_rad}"/> <!-- Original limit: 360 -->
+    <xacro:property name="j1_lower_limit" value="${-155 * deg_to_rad}"/> <!-- Original limit: -160 -->
+    <xacro:property name="j1_upper_limit" value="${155 * deg_to_rad}"/> <!-- Original limit: 160 -->
+    <xacro:property name="j2_lower_limit" value="${-20 * deg_to_rad}"/> <!-- Original limit: -25 -->
+    <xacro:property name="j2_upper_limit" value="${80 * deg_to_rad}"/> <!-- Original limit: 85 -->
+    <xacro:property name="j3_lower_limit" value="${-20 * deg_to_rad}"/> <!-- Original limit: -25 -->
+    <xacro:property name="j3_upper_limit" value="${100 * deg_to_rad}"/> <!-- Original limit: 105 -->
+    <xacro:property name="j4_lower_limit" value="${-355 * deg_to_rad}"/> <!-- Original limit: -360 -->
+    <xacro:property name="j4_upper_limit" value="${355 * deg_to_rad}"/> <!-- Original limit: 360 -->
     <!-- Velocity Limits (rad/s) -->
     <xacro:property name="j_velocity_limit" value="${300 * deg_to_rad}"/>
